Commit message: full body with control

File: description/kumi_core.xacro (robot description, xacro)
@@ -1,4 +1,3 @@
-<?xml version="1.0" ?>
-<robot xmlns:xacro="http://www.ros.org/wiki/xacro"  name="kumi">
+<robot xmlns:xacro="http://www.ros.org/wiki/xacro"  name="robot">
     <xacro:property name="thikness" value="0.3" />
     <xacro:property name="lenght" value="2" />
@@ -7,8 +6,7 @@
     <xacro:property name="toll" value="0.05" />
     <xacro:property name="mass" value="0.3" />
-    <xacro:property name="controller_yaml_path" value="/home/andreas/dev_ws/install/kumi_controller/share/kumi_controller/config/position_cntr.yaml" />
     <ros2_control name="KumiHardware" type="system">
         <hardware>
-        <plugin>gazebo_ros2_control/GazeboSystem</plugin>
+            <plugin>gazebo_ros2_control/GazeboSystem</plugin>
         </hardware>
         <joint name="front_sh">
@@ -28,4 +26,14 @@
         </joint>
         <joint name="back_knee">
+            <command_interface name="position"/>
+            <state_interface name="position"/>
+            <state_interface name="velocity"/>
+        </joint>
+        <joint name="front_ank">
+            <command_interface name="position"/>
+            <state_interface name="position"/>
+            <state_interface name="velocity"/>
+        </joint>
+        <joint name="back_ank">
             <command_interface name="position"/>
             <state_interface name="position"/>
@@ -38,4 +46,10 @@
         </plugin>
     </gazebo>
+    <link name="base_link"/>
+    <joint name="base_to_body" type="fixed">
+        <parent link="base_link"/>
+        <child link="body"/>
+        <origin xyz="0 0 0" rpy="0 0 0"/>
+    </joint>
     <link name="body">
         <visual>
@@ -44,6 +58,6 @@
                 <box size="${lenght} ${thikness} ${thikness}" />
             </geometry>
-            <material name="orange">
-                <color rgba="1 0.3 0.1 1"/>
+            <material name="green">
+                <color rgba="0.2 1 0.2 1"/>
             </material>
         </visual>
@@ -56,6 +70,6 @@
         <inertial>
             <origin xyz="0 0 0" rpy="0 0 0"/>
-            <mass value="12" />
-            <inertia ixx="2.26" ixy="0.0" ixz="0.0" iyy="6.26" iyz="0.0" izz="8.5" />
+            <mass value="1" />
+            <inertia ixx="0.015" ixy="0.0" ixz="0.0" iyy="0.340833" iyz="0.0" izz="0.340833" />
         </inertial>
     </link>
@@ -80,9 +94,9 @@
             </geometry>
             <material name="orange">
-                <color rgba="1 1 1 1"/>
-            </material>
-        </visual>
-        <collision>
-            <origin xyz="${thikness/2} 0 -${leg_len/4}" rpy="0 0 0"/>
+                <color rgba="0.2 1 0.2 1"/>
+            </material>
+        </visual>
+        <collision>
+            <origin xyz="${thikness/2} 0 ${-leg_len/4}" rpy="0 0 0"/>
             <geometry>
                 <box size="${thikness-toll} ${thikness-toll} ${leg_len/2-toll}" />
@@ -91,6 +105,6 @@
         <inertial>
             <origin xyz="${thikness/2} 0 ${-leg_len/4}" rpy="0 0 0"/>
-            <mass value="12" />
-            <inertia ixx="2.26" ixy="0.0" ixz="0.0" iyy="6.26" iyz="0.0" izz="8.5" />
+            <mass value="1" />
+            <inertia ixx="0.090833" ixy="0.0" ixz="0.0" iyy="0.090833" iyz="0.0" izz="0.015000" />
         </inertial>
     </link>
@@ -100,5 +114,5 @@
         <child link="front_leg_d"/>
         <axis xyz="0 0 1"/>
-        <limit lower="0" upper="0" velocity="100" effort="100"/>
+        <limit lower="${-pi/4}" upper="${pi/4}" velocity="100" effort="100"/>
     </joint>
     <transmission name="front_knee_trans">
@@ -130,4 +144,51 @@
         </inertial>
     </link>
+    <joint name="front_ank" type="revolute">
+        <origin xyz="0 0 ${-leg_len/2 - thikness/2}" rpy="0 0 0"/>
+        <parent link="front_leg_d"/>
+        <child link="front_foot"/>
+        <axis xyz="0 -1 0"/>
+        <limit lower="${-pi/8}" upper="${pi/8}" velocity="100" effort="100"/>
+    </joint>
+    <transmission name="front_ank_trans">
+        <type>transmission_interface/SimpleTransmission</type>
+        <actuator name="motor3">
+            <mechanicalReduction>1.0</mechanicalReduction>
+        </actuator>
+    </transmission>
+    <link name="front_foot">
+        <visual>
+            <origin xyz="0 0 0" rpy="0 0 0"/>
+            <geometry>
+                <box size="${foot_len} ${foot_len} ${thikness}" />
+            </geometry>
+            <material name="white">
+                <color rgba="0.2 1 0.2 1"/>
+            </material>
+        </visual>
+        <collision>
+            <origin xyz="0 0 0" rpy="0 0 0"/>
+            <geometry>
+                <box size="${foot_len} ${foot_len} ${thikness/2}" />
+            </geometry>
+        </collision>
+        <surface>
+            <friction>
+                <ode>
+                    <mu>1.0</mu>
+                    <mu2>1.0</mu2>
+                </ode>
+            </friction>
+        </surface>
+        <inertial>
+            <origin xyz="0 0 0" rpy="0 0 0"/>
+            <mass value="2" />
+            <inertia ixx="0.096667" ixy="0.0" ixz="0.0" iyy="0.096667" iyz="0.0" izz="0.163333" />
+        </inertial>
+    </link>
+    <gazebo reference="front_foot">
+        <mu1>10.0</mu1>
+        <mu2>10.0</mu2>
+    </gazebo>
     <joint name="back_sh" type="revolute">
         <origin xyz="${-lenght/2} 0 ${-thikness/2}" rpy="0 0 0"/>
@@ -165,5 +226,5 @@
         </inertial>
     </link>
-        <joint name="back_knee" type="revolute">
+    <joint name="back_knee" type="revolute">
         <origin xyz="${-thikness/2} 0 ${-leg_len/2}" rpy="0 0 0"/>
         <parent link="back_leg"/>
@@ -200,3 +261,46 @@
         </inertial>
     </link>
+    <joint name="back_ank" type="revolute">
+        <origin xyz="0 0 ${-leg_len/2 - thikness/2}" rpy="0 0 0"/>
+        <parent link="back_leg_d"/>
+        <child link="back_foot"/>
+        <axis xyz="0 -1 0"/>
+        <limit lower="-${pi/8}" upper="${pi/8}" velocity="100" effort="100"/>
+    </joint>
+    <transmission name="back_ank_trans">
+        <type>transmission_interface/SimpleTransmission</type>
+        <actuator name="motor6">
+            <mechanicalReduction>1.0</mechanicalReduction>
+        </actuator>
+    </transmission>
+    <link name="back_foot">
+        <visual>
+            <origin xyz="0 0 0" rpy="0 0 0"/>
+            <geometry>
+                <box size="${foot_len} ${foot_len} ${thikness}" />
+            </geometry>
+            <material name="white">
+                <color rgba="0.2 1 0.2 1"/>
+            </material>
+        </visual>
+        <collision>
+            <origin xyz="0 0 0" rpy="0 0 0"/>
+            <geometry>
+                <box size="${foot_len} ${foot_len} ${thikness/2}" />
+            </geometry>
+        </collision>
+        <surface>
+            <friction>
+                <ode>
+                    <mu>10.0</mu>
+                    <mu2>10.0</mu2>
+                </ode>
+            </friction>
+        </surface>
+        <inertial>
+            <origin xyz="0 0 0" rpy="0 0 0"/>
+            <mass value="2" />
+            <inertia ixx="0.096667" ixy="0.0" ixz="0.0" iyy="0.096667" iyz="0.0" izz="0.163333" />
+        </inertial>
+    </link>
 </robot>

Commit message: first controll

File: description/kumi_core.xacro (robot description, xacro)
@@ -46,10 +46,4 @@
         </plugin>
     </gazebo>
-    <link name="base_link"/>
-    <joint name="base_to_body" type="fixed">
-        <parent link="base_link"/>
-        <child link="body"/>
-        <origin xyz="0 0 0" rpy="0 0 0"/>
-    </joint>
     <link name="body">
         <visual>
@@ -70,5 +64,5 @@
         <inertial>
             <origin xyz="0 0 0" rpy="0 0 0"/>
-            <mass value="1" />
+            <mass value="0.1" />
             <inertia ixx="0.015" ixy="0.0" ixz="0.0" iyy="0.340833" iyz="0.0" izz="0.340833" />
         </inertial>
@@ -105,5 +99,5 @@
         <inertial>
             <origin xyz="${thikness/2} 0 ${-leg_len/4}" rpy="0 0 0"/>
-            <mass value="1" />
+            <mass value="0.1" />
             <inertia ixx="0.090833" ixy="0.0" ixz="0.0" iyy="0.090833" iyz="0.0" izz="0.015000" />
         </inertial>
@@ -140,5 +134,5 @@
         <inertial>
             <origin xyz="0 0 ${-leg_len/4}" rpy="0 0 0"/>
-            <mass value="1" />
+            <mass value="0.1" />
             <inertia ixx="0.090833" ixy="0.0" ixz="0.0" iyy="0.090833" iyz="0.0" izz="0.015000" />
         </inertial>
@@ -170,5 +164,5 @@
             <origin xyz="0 0 0" rpy="0 0 0"/>
             <geometry>
-                <box size="${foot_len} ${foot_len} ${thikness/2}" />
+                <box size="${foot_len} ${foot_len} ${thikness-toll}" />
             </geometry>
         </collision>
@@ -183,5 +177,5 @@
         <inertial>
             <origin xyz="0 0 0" rpy="0 0 0"/>
-            <mass value="2" />
+            <mass value="1" />
             <inertia ixx="0.096667" ixy="0.0" ixz="0.0" iyy="0.096667" iyz="0.0" izz="0.163333" />
         </inertial>
@@ -222,5 +216,5 @@
         <inertial>
             <origin xyz="${-thikness/2} 0 ${-leg_len/4}" rpy="0 0 0"/>
-            <mass value="1" />
+            <mass value="0.1" />
             <inertia ixx="0.090833" ixy="0.0" ixz="0.0" iyy="0.090833" iyz="0.0" izz="0.015000" />
         </inertial>
@@ -257,5 +251,5 @@
         <inertial>
             <origin xyz="0 0 ${-leg_len/4}" rpy="0 0 0"/>
-            <mass value="1" />
+            <mass value="0.1" />
             <inertia ixx="0.090833" ixy="0.0" ixz="0.0" iyy="0.090833" iyz="0.0" izz="0.015000" />
         </inertial>
@@ -287,5 +281,5 @@
             <origin xyz="0 0 0" rpy="0 0 0"/>
             <geometry>
-                <box size="${foot_len} ${foot_len} ${thikness/2}" />
+                <box size="${foot_len} ${foot_len} ${thikness-toll}" />
             </geometry>
         </collision>
@@ -300,5 +294,5 @@
         <inertial>
             <origin xyz="0 0 0" rpy="0 0 0"/>
-            <mass value="2" />
+            <mass value="1" />
             <inertia ixx="0.096667" ixy="0.0" ixz="0.0" iyy="0.096667" iyz="0.0" izz="0.163333" />
         </inertial>

Commit message: imu

File: description/kumi_core.xacro (robot description, xacro)
@@ -50,5 +50,5 @@
             <origin xyz="0 0 0" rpy="0 0 0"/>
             <geometry>
-                <box size="${lenght} ${thikness} ${thikness}" />
+                <box size="${lenght} ${thikness*2} ${thikness}" />
             </geometry>
             <material name="green">
@@ -59,19 +59,45 @@
             <origin xyz="0 0 0" rpy="0 0 0"/>
             <geometry>
-                <box size="${2-toll} ${thikness-toll} ${thikness-toll}" />
-            </geometry>
-        </collision>
-        <inertial>
-            <origin xyz="0 0 0" rpy="0 0 0"/>
-            <mass value="0.1" />
+                <box size="${lenght/1.5-toll} ${thikness*2-toll} ${thikness-toll}" />
+            </geometry>
+        </collision>
+        <inertial>
+            <origin xyz="0 0 0" rpy="0 0 0"/>
+            <mass value="1" />
             <inertia ixx="0.015" ixy="0.0" ixz="0.0" iyy="0.340833" iyz="0.0" izz="0.340833" />
         </inertial>
     </link>
+    <gazebo reference="body">
+        <sensor name="imu_sensor" type="imu">
+            <update_rate>20.0</update_rate>
+            <always_on>true</always_on>
+            <imu>
+            <angular_velocity>
+                <noise type="gaussian">
+                <mean>0.0</mean>
+                <stddev>0.1</stddev>
+                </noise>
+            </angular_velocity>
+            <linear_acceleration>
+                <noise type="gaussian">
+                <mean>0.0</mean>
+                <stddev>0.1</stddev>
+                </noise>
+            </linear_acceleration>
+            </imu>
+            <plugin name="imu_plugin" filename="libgazebo_ros_imu.so">
+            <ros>
+                <namespace>/</namespace>
+                <remapping>~/out:=/imu</remapping>
+            </ros>
+            </plugin>
+        </sensor>
+    </gazebo>
     <joint name="front_sh" type="revolute">
-        <origin xyz="${lenght/2} 0 ${-thikness/2}" rpy="0 0 0"/>
+        <origin xyz="${lenght/2+thikness/2} 0 0" rpy="0 0 0"/>
         <parent link="body"/>
         <child link="front_leg"/>
         <axis xyz="0 -1 0"/>
-        <limit lower="-${pi/4}" upper="${pi/2}" velocity="100" effort="100"/>
+        <limit lower="-${pi/2}" upper="${pi}" velocity="100" effort="100"/>
     </joint>
     <transmission name="front_sh_trans">
@@ -83,20 +109,20 @@
     <link name="front_leg">
         <visual>
+            <origin xyz="0 0 ${-leg_len/4 -thikness/2}" rpy="0 0 0"/>
+            <geometry>
+                <box size="${thikness} ${thikness*2} ${leg_len/2}" />
+            </geometry>
+            <material name="orange">
+                <color rgba="0.2 1 0.2 1"/>
+            </material>
+        </visual>
+        <collision>
+            <origin xyz="0 0 ${-leg_len/4 -thikness/2}" rpy="0 0 0"/>
+            <geometry>
+                <box size="${thikness-toll} ${thikness*2-toll} ${leg_len/2-toll}" />
+            </geometry>
+        </collision>
+        <inertial>
             <origin xyz="${thikness/2} 0 ${-leg_len/4}" rpy="0 0 0"/>
-            <geometry>
-                <box size="${thikness} ${thikness} ${leg_len/2}" />
-            </geometry>
-            <material name="orange">
-                <color rgba="0.2 1 0.2 1"/>
-            </material>
-        </visual>
-        <collision>
-            <origin xyz="${thikness/2} 0 ${-leg_len/4}" rpy="0 0 0"/>
-            <geometry>
-                <box size="${thikness-toll} ${thikness-toll} ${leg_len/2-toll}" />
-            </geometry>
-        </collision>
-        <inertial>
-            <origin xyz="${thikness/2} 0 ${-leg_len/4}" rpy="0 0 0"/>
             <mass value="0.1" />
             <inertia ixx="0.090833" ixy="0.0" ixz="0.0" iyy="0.090833" iyz="0.0" izz="0.015000" />
@@ -104,5 +130,5 @@
     </link>
     <joint name="front_knee" type="revolute">
-        <origin xyz="${thikness/2} 0 ${-leg_len/2}" rpy="0 0 0"/>
+        <origin xyz="0 0 ${-leg_len/2-thikness/2}" rpy="0 0 0"/>
         <parent link="front_leg"/>
         <child link="front_leg_d"/>
@@ -120,5 +146,5 @@
             <origin xyz="0 0 ${-leg_len/4}" rpy="0 0 0"/>
             <geometry>
-                <box size="${thikness} ${thikness} ${leg_len/2}" />
+                <box size="${thikness} ${thikness*2} ${leg_len/2}" />
             </geometry>
             <material name="orange">
@@ -129,5 +155,5 @@
             <origin xyz="0 0 ${-leg_len/4}" rpy="0 0 0"/>
             <geometry>
-                <box size="${thikness-toll} ${thikness-toll} ${leg_len/2-toll}" />
+                <box size="${thikness-toll} ${thikness*2-toll} ${leg_len/3-toll}" />
             </geometry>
         </collision>
@@ -143,5 +169,5 @@
         <child link="front_foot"/>
         <axis xyz="0 -1 0"/>
-        <limit lower="${-pi/8}" upper="${pi/8}" velocity="100" effort="100"/>
+        <limit lower="${-pi/2}" upper="${pi/2}" velocity="100" effort="100"/>
     </joint>
     <transmission name="front_ank_trans">
@@ -150,10 +176,10 @@
             <mechanicalReduction>1.0</mechanicalReduction>
         </actuator>
-    </transmission>
+    </transmission>0.0
     <link name="front_foot">
         <visual>
             <origin xyz="0 0 0" rpy="0 0 0"/>
             <geometry>
-                <box size="${foot_len} ${foot_len} ${thikness}" />
+                <box size="${foot_len+thikness} ${foot_len*2.5} ${thikness}" />
             </geometry>
             <material name="white">
@@ -164,5 +190,5 @@
             <origin xyz="0 0 0" rpy="0 0 0"/>
             <geometry>
-                <box size="${foot_len} ${foot_len} ${thikness-toll}" />
+                <box size="${foot_len+thikness} ${foot_len*2.5} ${thikness-toll}" />
             </geometry>
         </collision>
@@ -177,18 +203,20 @@
         <inertial>
             <origin xyz="0 0 0" rpy="0 0 0"/>
-            <mass value="1" />
-            <inertia ixx="0.096667" ixy="0.0" ixz="0.0" iyy="0.096667" iyz="0.0" izz="0.163333" />
+            <mass value="0.1" />
+            <inertia ixx="0.241667" ixy="0.0" ixz="0.0" iyy="0.454167" iyz="0.0" izz="0.163333" />
         </inertial>
     </link>
     <gazebo reference="front_foot">
-        <mu1>10.0</mu1>
-        <mu2>10.0</mu2>
+        <mu1>2</mu1>
+        <mu2>2</mu2>
+        <kp>1000000.0</kp>
+        <kd>100.0</kd>
     </gazebo>
     <joint name="back_sh" type="revolute">
-        <origin xyz="${-lenght/2} 0 ${-thikness/2}" rpy="0 0 0"/>
+        <origin xyz="${-lenght/2-thikness/2} 0 0" rpy="0 0 0"/>
         <parent link="body"/>
         <child link="back_leg"/>
         <axis xyz="0 -1 0"/>
-        <limit lower="-${pi/2}" upper="${pi/4}" velocity="100" effort="100"/>
+        <limit lower="-${1.5*pi}" upper="${pi/2}" velocity="100" effort="100"/>
     </joint>
     <transmission name="back_sh_trans">
@@ -200,20 +228,20 @@
     <link name="back_leg">
         <visual>
+            <origin xyz="0 0 ${-leg_len/4 -thikness/2}" rpy="0 0 0"/>
+            <geometry>
+                <box size="${thikness} ${thikness*2} ${leg_len/2}" />
+            </geometry>
+            <material name="orange">
+                <color rgba="0.2 1 0.2 1"/>
+            </material>
+        </visual>
+        <collision>
+            <origin xyz="0 0 ${-leg_len/4 -thikness/2}" rpy="0 0 0"/>
+            <geometry>
+                <box size="${thikness-toll} ${thikness*2-toll} ${leg_len/2-toll}" />
+            </geometry>
+        </collision>
+        <inertial>
             <origin xyz="${-thikness/2} 0 ${-leg_len/4}" rpy="0 0 0"/>
-            <geometry>
-                <box size="${thikness} ${thikness} ${leg_len/2}" />
-            </geometry>
-            <material name="orange">
-                <color rgba="0.2 1 0.2 1"/>
-            </material>
-        </visual>
-        <collision>
-            <origin xyz="${-thikness/2} 0 ${-leg_len/4}" rpy="0 0 0"/>
-            <geometry>
-                <box size="${thikness-toll} ${thikness-toll} ${leg_len/2-toll}" />
-            </geometry>
-        </collision>
-        <inertial>
-            <origin xyz="${-thikness/2} 0 ${-leg_len/4}" rpy="0 0 0"/>
             <mass value="0.1" />
             <inertia ixx="0.090833" ixy="0.0" ixz="0.0" iyy="0.090833" iyz="0.0" izz="0.015000" />
@@ -221,5 +249,5 @@
     </link>
     <joint name="back_knee" type="revolute">
-        <origin xyz="${-thikness/2} 0 ${-leg_len/2}" rpy="0 0 0"/>
+        <origin xyz="0 0 ${-leg_len/2 -thikness/2}" rpy="0 0 0"/>
         <parent link="back_leg"/>
         <child link="back_leg_d"/>
@@ -237,5 +265,5 @@
             <origin xyz="0 0 ${-leg_len/4}" rpy="0 0 0"/>
             <geometry>
-                <box size="${thikness} ${thikness} ${leg_len/2}" />
+                <box size="${thikness} ${thikness*2} ${leg_len/2}" />
             </geometry>
             <material name="orange">
@@ -246,5 +274,5 @@
             <origin xyz="0 0 ${-leg_len/4}" rpy="0 0 0"/>
             <geometry>
-                <box size="${thikness-toll} ${thikness-toll} ${leg_len/2-toll}" />
+                <box size="${thikness-toll} ${thikness*2-toll} ${leg_len/3-toll}" />
             </geometry>
         </collision>
@@ -260,5 +288,5 @@
         <child link="back_foot"/>
         <axis xyz="0 -1 0"/>
-        <limit lower="-${pi/8}" upper="${pi/8}" velocity="100" effort="100"/>
+        <limit lower="-${pi/2}" upper="${pi/2}" velocity="100" effort="100"/>
     </joint>
     <transmission name="back_ank_trans">
@@ -272,5 +300,5 @@
             <origin xyz="0 0 0" rpy="0 0 0"/>
             <geometry>
-                <box size="${foot_len} ${foot_len} ${thikness}" />
+                <box size="${foot_len+thikness} ${foot_len*2.5} ${thikness}" />
             </geometry>
             <material name="white">
@@ -281,20 +309,18 @@
             <origin xyz="0 0 0" rpy="0 0 0"/>
             <geometry>
-                <box size="${foot_len} ${foot_len} ${thikness-toll}" />
-            </geometry>
-        </collision>
-        <surface>
-            <friction>
-                <ode>
-                    <mu>10.0</mu>
-                    <mu2>10.0</mu2>
-                </ode>
-            </friction>
-        </surface>
-        <inertial>
-            <origin xyz="0 0 0" rpy="0 0 0"/>
-            <mass value="1" />
-            <inertia ixx="0.096667" ixy="0.0" ixz="0.0" iyy="0.096667" iyz="0.0" izz="0.163333" />
-        </inertial>
-    </link>
+                <box size="${foot_len+thikness} ${foot_len*2.5} ${thikness-toll}" />
+            </geometry>
+        </collision>
+        <inertial>
+            <origin xyz="0 0 0" rpy="0 0 0"/>
+            <mass value="0.1" />
+            <inertia ixx="0.241667" ixy="0.0" ixz="0.0" iyy="0.454167" iyz="0.0" izz="0.163333" />
+        </inertial>
+    </link>
+     <gazebo reference="back_foot">
+        <mu1>2</mu1>
+        <mu2>2</mu2>
+        <kp>1000000.0</kp>
+        <kd>100.0</kd>
+    </gazebo>
 </robot>

Commit message: imu pluing installed (working)

File: description/kumi_core.xacro (robot description, xacro)
@@ -1,8 +1,8 @@
 <robot xmlns:xacro="http://www.ros.org/wiki/xacro"  name="robot">
-    <xacro:property name="thikness" value="0.3" />
-    <xacro:property name="lenght" value="2" />
-    <xacro:property name="leg_len" value="1.5" />
-    <xacro:property name="foot_len" value="0.7" />
-    <xacro:property name="toll" value="0.05" />
+    <xacro:property name="thikness" value="0.15" />
+    <xacro:property name="lenght" value="0.5" />
+    <xacro:property name="leg_len" value="0.5" />
+    <xacro:property name="foot_len" value="0.2" />
+    <xacro:property name="toll" value="0.005" />
     <xacro:property name="mass" value="0.3" />
     <ros2_control name="KumiHardware" type="system">
@@ -50,5 +50,5 @@
             <origin xyz="0 0 0" rpy="0 0 0"/>
             <geometry>
-                <box size="${lenght} ${thikness*2} ${thikness}" />
+                <box size="${lenght+2*thikness} ${thikness*2} ${thikness}" />
             </geometry>
             <material name="green">
@@ -86,5 +86,5 @@
             </linear_acceleration>
             </imu>
-            <plugin name="imu_plugin" filename="libgazebo_ros_imu.so">
+            <plugin filename="libgazebo_ros_imu_sensor.so" name="imu_sensor">
             <ros>
                 <namespace>/</namespace>
