Commit message: effort controller non funzionante

File: description/kumi_core.xacro (robot description, xacro)
@@ -46,4 +46,14 @@
         </plugin>
     </gazebo>
+    <physics type="ode">
+    <max_step_size>0.001</max_step_size>
+    <real_time_update_rate>1000</real_time_update_rate>
+    <ode>
+        <solver>
+        <iters>50</iters>
+        <sor>1.3</sor>
+        </solver>
+    </ode>
+    </physics>
     <link name="body">
         <visual>
@@ -64,5 +74,5 @@
         <inertial>
             <origin xyz="0 0 0" rpy="0 0 0"/>
-            <mass value="1" />
+            <mass value="0.5" />
             <inertia ixx="0.015" ixy="0.0" ixz="0.0" iyy="0.340833" iyz="0.0" izz="0.340833" />
         </inertial>
@@ -125,5 +135,5 @@
         <inertial>
             <origin xyz="${thikness/2} 0 ${-leg_len/4}" rpy="0 0 0"/>
-            <mass value="0.1" />
+            <mass value="0.3" />
             <inertia ixx="0.090833" ixy="0.0" ixz="0.0" iyy="0.090833" iyz="0.0" izz="0.015000" />
         </inertial>
@@ -160,5 +170,5 @@
         <inertial>
             <origin xyz="0 0 ${-leg_len/4}" rpy="0 0 0"/>
-            <mass value="0.1" />
+            <mass value="0.3" />
             <inertia ixx="0.090833" ixy="0.0" ixz="0.0" iyy="0.090833" iyz="0.0" izz="0.015000" />
         </inertial>
@@ -169,5 +179,5 @@
         <child link="front_foot"/>
         <axis xyz="0 -1 0"/>
-        <limit lower="${-pi/2}" upper="${pi/2}" velocity="100" effort="100"/>
+        <limit lower="${-pi/4}" upper="${pi/4}" velocity="100" effort="100"/>
     </joint>
     <transmission name="front_ank_trans">
@@ -181,5 +191,5 @@
             <origin xyz="0 0 0" rpy="0 0 0"/>
             <geometry>
-                <box size="${foot_len+thikness} ${foot_len*2.5} ${thikness}" />
+                <box size="${foot_len+thikness} ${foot_len*2.5} ${thikness-toll}" />
             </geometry>
             <material name="white">
@@ -193,24 +203,10 @@
             </geometry>
         </collision>
-        <surface>
-            <friction>
-                <ode>
-                    <mu>1.0</mu>
-                    <mu2>1.0</mu2>
-                </ode>
-            </friction>
-        </surface>
-        <inertial>
-            <origin xyz="0 0 0" rpy="0 0 0"/>
-            <mass value="0.1" />
+        <inertial>
+            <origin xyz="0 0 0" rpy="0 0 0"/>
+            <mass value="0.2" />
             <inertia ixx="0.241667" ixy="0.0" ixz="0.0" iyy="0.454167" iyz="0.0" izz="0.163333" />
         </inertial>
     </link>
-    <gazebo reference="front_foot">
-        <mu1>2</mu1>
-        <mu2>2</mu2>
-        <kp>1000000.0</kp>
-        <kd>100.0</kd>
-    </gazebo>
     <joint name="back_sh" type="revolute">
         <origin xyz="${-lenght/2-thikness/2} 0 0" rpy="0 0 0"/>
@@ -244,5 +240,5 @@
         <inertial>
             <origin xyz="${-thikness/2} 0 ${-leg_len/4}" rpy="0 0 0"/>
-            <mass value="0.1" />
+            <mass value="0.3" />
             <inertia ixx="0.090833" ixy="0.0" ixz="0.0" iyy="0.090833" iyz="0.0" izz="0.015000" />
         </inertial>
@@ -279,5 +275,5 @@
         <inertial>
             <origin xyz="0 0 ${-leg_len/4}" rpy="0 0 0"/>
-            <mass value="0.1" />
+            <mass value="0.3" />
             <inertia ixx="0.090833" ixy="0.0" ixz="0.0" iyy="0.090833" iyz="0.0" izz="0.015000" />
         </inertial>
@@ -288,5 +284,5 @@
         <child link="back_foot"/>
         <axis xyz="0 -1 0"/>
-        <limit lower="-${pi/2}" upper="${pi/2}" velocity="100" effort="100"/>
+        <limit lower="-${pi/4}" upper="${pi/4}" velocity="100" effort="100"/>
     </joint>
     <transmission name="back_ank_trans">
@@ -300,5 +296,5 @@
             <origin xyz="0 0 0" rpy="0 0 0"/>
             <geometry>
-                <box size="${foot_len+thikness} ${foot_len*2.5} ${thikness}" />
+                <box size="${foot_len+thikness} ${foot_len*2.5} ${thikness-toll}" />
             </geometry>
             <material name="white">
@@ -314,13 +310,7 @@
         <inertial>
             <origin xyz="0 0 0" rpy="0 0 0"/>
-            <mass value="0.1" />
+            <mass value="0.2" />
             <inertia ixx="0.241667" ixy="0.0" ixz="0.0" iyy="0.454167" iyz="0.0" izz="0.163333" />
         </inertial>
     </link>
-     <gazebo reference="back_foot">
-        <mu1>2</mu1>
-        <mu2>2</mu2>
-        <kp>1000000.0</kp>
-        <kd>100.0</kd>
-    </gazebo>
 </robot>

File: description/kumi_easy.xacro (robot description, xacro)
@@ -7,45 +7,4 @@
     <xacro:property name="toll" value="0.005" />
     <xacro:property name="mass" value="0.3" />
-    <xacro:property name="controller_yaml_path" value="/home/andreas/dev_ws/install/kumi_controller/share/kumi_controller/config/position_cntr.yaml" />
-    <ros2_control name="KumiHardware" type="system">
-        <hardware>
-            <plugin>gazebo_ros2_control/GazeboSystem</plugin>
-        </hardware>
-        <joint name="front_sh">
-            <command_interface name="position"/>
-            <state_interface name="position"/>
-            <state_interface name="velocity"/>
-        </joint>
-        <joint name="back_sh">
-            <command_interface name="position"/>
-            <state_interface name="position"/>
-            <state_interface name="velocity"/>
-        </joint>
-        <joint name="front_knee">
-            <command_interface name="position"/>
-            <state_interface name="position"/>
-            <state_interface name="velocity"/>
-        </joint>
-        <joint name="back_knee">
-            <command_interface name="position"/>
-            <state_interface name="position"/>
-            <state_interface name="velocity"/>
-        </joint>
-        <joint name="front_ank">
-            <command_interface name="position"/>
-            <state_interface name="position"/>
-            <state_interface name="velocity"/>
-        </joint>
-        <joint name="back_ank">
-            <command_interface name="position"/>
-            <state_interface name="position"/>
-            <state_interface name="velocity"/>
-        </joint>
-    </ros2_control>
-    <gazebo>
-        <plugin name="gazebo_ros2_control" filename="libgazebo_ros2_control.so">
-            <parameters>/home/andreas/dev_ws/install/kumi_controller/share/kumi_controller/config/kumi_control_config.yaml</parameters>
-        </plugin>
-    </gazebo>s
     <link name="body">
         <visual>
@@ -75,12 +34,6 @@
         <child link="front_leg"/>
         <axis xyz="0 -1 0"/>
-        <limit lower="-${pi/2}" upper="${pi}" velocity="100" effort="100"/>
-    </joint>
-    <transmission name="front_sh_trans">
-        <type>transmission_interface/SimpleTransmission</type>
-        <actuator name="motor1">
-            <mechanicalReduction>1.0</mechanicalReduction>
-        </actuator>
-    </transmission>
+        <limit lower="0" upper="0" velocity="100" effort="100"/>
+    </joint>
     <link name="front_leg">
         <visual>
@@ -110,12 +63,6 @@
         <child link="front_leg_d"/>
         <axis xyz="0 0 1"/>
-        <limit lower="${-pi/4}" upper="${pi/4}" velocity="100" effort="100"/>
-    </joint>
-    <transmission name="front_knee_trans">
-        <type>transmission_interface/SimpleTransmission</type>
-        <actuator name="motor2">
-            <mechanicalReduction>1.0</mechanicalReduction>
-        </actuator>
-    </transmission>
+        <limit lower="0" upper="0" velocity="100" effort="100"/>
+    </joint>
     <link name="front_leg_d">
         <visual>
@@ -145,12 +92,6 @@
         <child link="front_foot"/>
         <axis xyz="0 -1 0"/>
-        <limit lower="${-pi/4}" upper="${pi/4}" velocity="100" effort="100"/>
-    </joint>
-    <transmission name="front_ank_trans">
-        <type>transmission_interface/SimpleTransmission</type>
-        <actuator name="motor3">
-            <mechanicalReduction>1.0</mechanicalReduction>
-        </actuator>
-    </transmission>
+        <limit lower="0" upper="0" velocity="100" effort="100"/>
+    </joint>
     <link name="front_foot">
         <visual>
@@ -180,12 +121,6 @@
         <child link="back_leg"/>
         <axis xyz="0 -1 0"/>
-        <limit lower="-${pi}" upper="${pi/2}" velocity="100" effort="100"/>
-    </joint>
-    <transmission name="back_sh_trans">
-        <type>transmission_interface/SimpleTransmission</type>
-        <actuator name="motor4">
-            <mechanicalReduction>1.0</mechanicalReduction>
-        </actuator>
-    </transmission>
+        <limit lower="0" upper="0" velocity="100" effort="100"/>
+    </joint>
     <link name="back_leg">
         <visual>
@@ -215,12 +150,6 @@
         <child link="back_leg_d"/>
         <axis xyz="0 0 1"/>
-        <limit lower="${-pi/4}" upper="${pi/4}" velocity="100" effort="100"/>
-    </joint>
-    <transmission name="back_knee_trans">
-        <type>transmission_interface/SimpleTransmission</type>
-        <actuator name="motor5">
-            <mechanicalReduction>1.0</mechanicalReduction>
-        </actuator>
-    </transmission>
+        <limit lower="0" upper="0" velocity="100" effort="100"/>
+    </joint>
     <link name="back_leg_d">
         <visual>
@@ -250,12 +179,6 @@
         <child link="back_foot"/>
         <axis xyz="0 -1 0"/>
-        <limit lower="${-pi/4}" upper="${pi/4}" velocity="100" effort="100"/>
-    </joint>
-    <transmission name="back_ank_trans">
-        <type>transmission_interface/SimpleTransmission</type>
-        <actuator name="motor6">
-            <mechanicalReduction>1.0</mechanicalReduction>
-        </actuator>
-    </transmission>
+        <limit lower="0" upper="0" velocity="100" effort="100"/>
+    </joint>
     <link name="back_foot">
         <visual>
