Commit message: updated yaml

File: description/kumi.xacro (robot description, xacro)
@@ -1,9 +1,9 @@
-<robot xmlns:xacro="http://www.ros.org/wiki/xacro"  name="robot">
-    <!-- Variables -->
+<?xml version="1.0" ?>
+<robot xmlns:xacro="http://www.ros.org/wiki/xacro"  name="kumi">
     <xacro:property name="thikness" value="0.3" />
     <xacro:property name="lenght" value="2" />
     <xacro:property name="leg_len" value="1.5" />
     <xacro:property name="foot_len" value="0.7" />
-    <!-- Specify some colours -->
+    <xacro:property name="controller_yaml_path" value="/home/andreas/dev_ws/install/kumi_controller/share/kumi_controller/config/position_cntr.yaml" />
     <material name="white">
         <color rgba="1 1 1 1"/>
@@ -15,6 +15,4 @@
         <color rgba="0.2 0.2 1 1"/>
     </material>
-    <!-- Specify some standard inertial calculations https://en.wikipedia.org/wiki/List_of_moments_of_inertia -->
-    <!-- These make use of xacro's mathematical functionality -->
     <xacro:macro name="inertial_sphere" params="mass radius *origin">
         <inertial>
@@ -44,9 +42,4 @@
         </inertial>
     </xacro:macro>
-    <!-- base_link is a large rectangular plate. Some things to note: -->
-    <!-- - We set the visual origin Z to half the box height, so that the link origin sits at the bottom of the box -->
-    <!-- - We set the collision to be identical to the visual -->
-    <!-- - We specified the colour manually (but still need to enter a name) -->
-    <!-- - We specified all the inertial parameters manually -->
     <link name="body">
         <visual>
@@ -71,8 +64,4 @@
         </inertial>
     </link>
-    <!-- slider_joint lets slider_link move back and forth along the top of the base in one dimension.  -->
-    <!-- - Origin is set to one of the top edges of the base_link box, so that our link skims across the top  -->
-    <!-- - It moves along the X axis -->
-    <!-- - We need to specify limits for the motion -->
     <joint name="front_sh" type="revolute">
         <origin xyz="${lenght/2} 0 ${-thikness/2}" rpy="0 0 0"/>
@@ -84,10 +73,8 @@
     <transmission name="front_sh_trans">
         <type>transmission_interface/SimpleTransmission</type>
-        <joint name="front_sh"/>
         <actuator name="motor1">
             <mechanicalReduction>1.0</mechanicalReduction>
         </actuator>
     </transmission>
-  <!-- ros2_control interface -->
   <ros2_control name="KumiHardware" type="system">
     <hardware>
@@ -100,9 +87,9 @@
     </joint>
   </ros2_control>
-    <!-- base_link is a large rectangular plate. Some things to note: -->
-    <!-- - We set the visual origin Z to half the box height, so that the link origin sits at the bottom of the box -->
-    <!-- - We set the collision to be identical to the visual -->
-    <!-- - We specified the colour manually (but still need to enter a name) -->
-    <!-- - We specified all the inertial parameters manually -->
+  <gazebo>
+    <plugin name="gazebo_ros2_control" filename="libgazebo_ros2_control.so">
+        <parameters>/home/andreas/dev_ws/install/kumi_controller/share/kumi_controller/config/kumi_control_config.yaml</parameters>
+    </plugin>
+  </gazebo>
     <link name="front_leg">
         <visual>
@@ -127,4 +114,3 @@
         </inertial>
     </link>
-        <!-- This file is not a robot in and of itself, it just contains some useful tags that could be included in any robot -->
 </robot>

Commit message: name change

File: description/kumi.xacro (robot description, xacro)
@@ -7,5 +7,4 @@
     <xacro:property name="toll" value="0.005" />
     <xacro:property name="mass" value="0.3" />
-    <xacro:property name="controller_yaml_path" value="/home/andreas/dev_ws/install/kumi_controller/share/kumi_controller/config/position_cntr.yaml" />
     <ros2_control name="KumiHardware" type="system">
         <hardware>
@@ -13,30 +12,36 @@
         </hardware>
         <joint name="front_sh">
-            <command_interface name="position"/>
+            <command_interface name="effort"/>
+            <state_interface name="effort"/>
             <state_interface name="position"/>
             <state_interface name="velocity"/>
         </joint>
         <joint name="back_sh">
-            <command_interface name="position"/>
+            <command_interface name="effort"/>
+            <state_interface name="effort"/>
             <state_interface name="position"/>
             <state_interface name="velocity"/>
         </joint>
         <joint name="front_knee">
-            <command_interface name="position"/>
+            <command_interface name="effort"/>
+            <state_interface name="effort"/>
             <state_interface name="position"/>
             <state_interface name="velocity"/>
         </joint>
         <joint name="back_knee">
-            <command_interface name="position"/>
+            <command_interface name="effort"/>
+            <state_interface name="effort"/>
             <state_interface name="position"/>
             <state_interface name="velocity"/>
         </joint>
         <joint name="front_ank">
-            <command_interface name="position"/>
+            <command_interface name="effort"/>
+            <state_interface name="effort"/>
             <state_interface name="position"/>
             <state_interface name="velocity"/>
         </joint>
         <joint name="back_ank">
-            <command_interface name="position"/>
+            <command_interface name="effort"/>
+            <state_interface name="effort"/>
             <state_interface name="position"/>
             <state_interface name="velocity"/>
@@ -45,5 +50,5 @@
     <gazebo>
         <plugin name="gazebo_ros2_control" filename="libgazebo_ros2_control.so">
-            <parameters>/home/andreas/dev_ws/install/kumi_controller/share/kumi_controller/config/kumi_control_config.yaml</parameters>
+            <parameters>/home/andreas/dev_ws/install/kumi/share/kumi/config/kumi_effort_cntr_cnfg.yaml</parameters>
         </plugin>
     </gazebo>s
@@ -77,10 +82,4 @@
         <limit lower="-${pi/2}" upper="${pi}" velocity="100" effort="100"/>
     </joint>
-    <transmission name="front_sh_trans">
-        <type>transmission_interface/SimpleTransmission</type>
-        <actuator name="motor1">
-            <mechanicalReduction>1.0</mechanicalReduction>
-        </actuator>
-    </transmission>
     <link name="front_leg">
         <visual>
@@ -112,10 +111,4 @@
         <limit lower="${-pi/4}" upper="${pi/4}" velocity="100" effort="100"/>
     </joint>
-    <transmission name="front_knee_trans">
-        <type>transmission_interface/SimpleTransmission</type>
-        <actuator name="motor2">
-            <mechanicalReduction>1.0</mechanicalReduction>
-        </actuator>
-    </transmission>
     <link name="front_leg_d">
         <visual>
@@ -147,10 +140,4 @@
         <limit lower="${-pi/4}" upper="${pi/4}" velocity="100" effort="100"/>
     </joint>
-    <transmission name="front_ank_trans">
-        <type>transmission_interface/SimpleTransmission</type>
-        <actuator name="motor3">
-            <mechanicalReduction>1.0</mechanicalReduction>
-        </actuator>
-    </transmission>
     <link name="front_foot">
         <visual>
@@ -182,10 +169,4 @@
         <limit lower="-${pi}" upper="${pi/2}" velocity="100" effort="100"/>
     </joint>
-    <transmission name="back_sh_trans">
-        <type>transmission_interface/SimpleTransmission</type>
-        <actuator name="motor4">
-            <mechanicalReduction>1.0</mechanicalReduction>
-        </actuator>
-    </transmission>
     <link name="back_leg">
         <visual>
@@ -217,10 +198,4 @@
         <limit lower="${-pi/4}" upper="${pi/4}" velocity="100" effort="100"/>
     </joint>
-    <transmission name="back_knee_trans">
-        <type>transmission_interface/SimpleTransmission</type>
-        <actuator name="motor5">
-            <mechanicalReduction>1.0</mechanicalReduction>
-        </actuator>
-    </transmission>
     <link name="back_leg_d">
         <visual>
@@ -252,10 +227,4 @@
         <limit lower="${-pi/4}" upper="${pi/4}" velocity="100" effort="100"/>
     </joint>
-    <transmission name="back_ank_trans">
-        <type>transmission_interface/SimpleTransmission</type>
-        <actuator name="motor6">
-            <mechanicalReduction>1.0</mechanicalReduction>
-        </actuator>
-    </transmission>
     <link name="back_foot">
         <visual>

File: description/kumi_core.xacro (robot description, xacro)
@@ -43,5 +43,5 @@
     <gazebo>
         <plugin name="gazebo_ros2_control" filename="libgazebo_ros2_control.so">
-            <parameters>/home/andreas/dev_ws/install/kumi_controller/share/kumi_controller/config/kumi_control_config.yaml</parameters>
+            <parameters>/home/andreas/dev_ws/install/kumi_controller/share/kumi_controller/config/kumi_effort_cntr_cnfg.yaml</parameters>
         </plugin>
     </gazebo>

Commit message: effort_controller, PID not tuned starting to connect matlab

File: description/kumi.xacro (robot description, xacro)
@@ -7,4 +7,5 @@
     <xacro:property name="toll" value="0.005" />
     <xacro:property name="mass" value="0.3" />
+    <xacro:property name="joint_friction" value="0.5" />
     <ros2_control name="KumiHardware" type="system">
         <hardware>
@@ -80,5 +81,6 @@
         <child link="front_leg"/>
         <axis xyz="0 -1 0"/>
-        <limit lower="-${pi/2}" upper="${pi}" velocity="100" effort="100"/>
+        <limit lower="-0.5" upper="0.5" velocity="5" effort="2"/>
+        <dynamics damping="0.1" friction="${joint_friction}"/>
     </joint>
     <link name="front_leg">
@@ -109,5 +111,6 @@
         <child link="front_leg_d"/>
         <axis xyz="0 0 1"/>
-        <limit lower="${-pi/4}" upper="${pi/4}" velocity="100" effort="100"/>
+        <limit lower="-0.5" upper="0.5" velocity="5" effort="2"/>
+        <dynamics damping="10.0" friction="10.0"/>
     </joint>
     <link name="front_leg_d">
@@ -138,5 +141,6 @@
         <child link="front_foot"/>
         <axis xyz="0 -1 0"/>
-        <limit lower="${-pi/4}" upper="${pi/4}" velocity="100" effort="100"/>
+        <limit lower="-0.5" upper="0.5" velocity="5" effort="2"/>
+        <dynamics damping="0.1" friction="${joint_friction}"/>
     </joint>
     <link name="front_foot">
@@ -167,5 +171,6 @@
         <child link="back_leg"/>
         <axis xyz="0 -1 0"/>
-        <limit lower="-${pi}" upper="${pi/2}" velocity="100" effort="100"/>
+        <limit lower="-0.5" upper="0.5" velocity="5" effort="2"/>
+        <dynamics damping="0.1" friction="${joint_friction}"/>
     </joint>
     <link name="back_leg">
@@ -196,5 +201,6 @@
         <child link="back_leg_d"/>
         <axis xyz="0 0 1"/>
-        <limit lower="${-pi/4}" upper="${pi/4}" velocity="100" effort="100"/>
+        <limit lower="-0.5" upper="0.5" velocity="5" effort="2"/>
+        <dynamics damping="10.0" friction="10.0"/>
     </joint>
     <link name="back_leg_d">
@@ -225,5 +231,6 @@
         <child link="back_foot"/>
         <axis xyz="0 -1 0"/>
-        <limit lower="${-pi/4}" upper="${pi/4}" velocity="100" effort="100"/>
+        <limit lower="-0.5" upper="0.5" velocity="5" effort="2"/>
+        <dynamics damping="0.1" friction="${joint_friction}"/>
     </joint>
     <link name="back_foot">

Commit message: GUI not working

File: description/kumi.xacro (robot description, xacro)
@@ -73,5 +73,5 @@
             <origin xyz="0 0 0" rpy="0 0 0"/>
             <mass value="0.5" />
-            <inertia ixx="0.015" ixy="0.0" ixz="0.0" iyy="0.340833" iyz="0.0" izz="0.340833" />
+            <inertia ixx="0.001875" ixy="0.0" ixz="0.0" iyy="0.011354" iyz="0.0" izz="0.011354" />
         </inertial>
     </link>
@@ -103,5 +103,5 @@
             <origin xyz="0 0 ${-leg_len/2}" rpy="0 0 0"/>
             <mass value="0.3" />
-            <inertia ixx="0.090833" ixy="0.0" ixz="0.0" iyy="0.090833" iyz="0.0" izz="0.015000" />
+            <inertia ixx="0.001562" ixy="0.0" ixz="0.0" iyy="0.001562" iyz="0.0" izz="0.001125" />
         </inertial>
     </link>
@@ -133,5 +133,5 @@
             <origin xyz="0 0 0" rpy="0 0 0"/>
             <mass value="0.3" />
-            <inertia ixx="0.090833" ixy="0.0" ixz="0.0" iyy="0.090833" iyz="0.0" izz="0.015000" />
+            <inertia ixx="0.001562" ixy="0.0" ixz="0.0" iyy="0.001562" iyz="0.0" izz="0.001125" />
         </inertial>
     </link>
@@ -163,5 +163,5 @@
             <origin xyz="0 0 0" rpy="0 0 0"/>
             <mass value="0.2" />
-            <inertia ixx="0.241667" ixy="0.0" ixz="0.0" iyy="0.454167" iyz="0.0" izz="0.163333" />
+            <inertia ixx="0.001135" ixy="0.0" ixz="0.0" iyy="0.001135" iyz="0.0" izz="0.002083" />
         </inertial>
     </link>
@@ -193,5 +193,5 @@
             <origin xyz="0 0 ${-leg_len/2}" rpy="0 0 0"/>
             <mass value="0.3" />
-            <inertia ixx="0.090833" ixy="0.0" ixz="0.0" iyy="0.090833" iyz="0.0" izz="0.015000" />
+            <inertia ixx="0.001562" ixy="0.0" ixz="0.0" iyy="0.001562" iyz="0.0" izz="0.001125" />
         </inertial>
     </link>
@@ -223,5 +223,5 @@
             <origin xyz="0 0 0" rpy="0 0 0"/>
             <mass value="0.3" />
-            <inertia ixx="0.090833" ixy="0.0" ixz="0.0" iyy="0.090833" iyz="0.0" izz="0.015000" />
+            <inertia ixx="0.001562" ixy="0.0" ixz="0.0" iyy="0.001562" iyz="0.0" izz="0.001125" />
         </inertial>
     </link>
@@ -253,5 +253,5 @@
             <origin xyz="0 0 0" rpy="0 0 0"/>
             <mass value="0.2" />
-            <inertia ixx="0.241667" ixy="0.0" ixz="0.0" iyy="0.454167" iyz="0.0" izz="0.163333" />
+            <inertia ixx="0.001135" ixy="0.0" ixz="0.0" iyy="0.001135" iyz="0.0" izz="0.002083" />
         </inertial>
     </link>
